Commit message: 2

File: src/slam_nav/urdf/ugv_rover.urdf (robot description, URDF)
Before this commit: robot ugv_rover, 13 links, 12 joints
Links:
- link 3d_camera_link: geometry collision mesh filename=package://slam_nav/meshes/ugv_rover/3d_camera_link.stl; visual mesh filename=package://slam_nav/meshes/ugv_rover/3d_camera_link.stl
- link base_lidar_link: geometry collision mesh filename=package://slam_nav/meshes/ugv_rover/base_lidar_link.stl; visual mesh filename=package://slam_nav/meshes/ugv_rover/base_lidar_link.stl
- link base_link: geometry collision mesh filename=package://slam_nav/meshes/ugv_rover/base_link.stl; visual mesh filename=package://slam_nav/meshes/ugv_rover/base_link.stl
- link left_down_wheel_link: geometry collision mesh filename=package://slam_nav/meshes/ugv_rover/left_down_wheel_link.stl; visual mesh filename=package://slam_nav/meshes/ugv_rover/left_down_wheel_link.stl
- link left_up_wheel_link: geometry collision mesh filename=package://slam_nav/meshes/ugv_rover/left_up_wheel_link.stl; visual mesh filename=package://slam_nav/meshes/ugv_rover/left_up_wheel_link.stl
- link pt_base_link: geometry collision mesh filename=package://slam_nav/meshes/ugv_rover/pt_base_link.stl; visual mesh filename=package://slam_nav/meshes/ugv_rover/pt_base_link.stl
- link pt_camera_link: geometry collision mesh filename=package://slam_nav/meshes/ugv_rover/pt_camera_link.stl; visual mesh filename=package://slam_nav/meshes/ugv_rover/pt_camera_link.stl
- link pt_link1: geometry collision mesh filename=package://slam_nav/meshes/ugv_rover/pt_link1.stl; visual mesh filename=package://slam_nav/meshes/ugv_rover/pt_link1.stl
- link pt_link2: geometry collision mesh filename=package://slam_nav/meshes/ugv_rover/pt_link2.stl; visual mesh filename=package://slam_nav/meshes/ugv_rover/pt_link2.stl
- link right_down_wheel_link: geometry collision mesh filename=package://slam_nav/meshes/ugv_rover/right_down_wheel_link.s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; visual mesh filename=package://slam_nav/meshes/ugv_rover/right_down_wheel_link.s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
- link right_up_wheel_link: geometry collision mesh filename=package://slam_nav/meshes/ugv_rover/right_up_wheel_link.stl; visual mesh filename=package://slam_nav/meshes/ugv_rover/right_up_wheel_link.stl
